File: pcb/panelize/panelize.kicad_pcb (KiCad board)
At the start: 2 copper layers, 96 x 92.5 mm, 600 parts, among them J1 Conn_01x05_Pin, J2 Conn_01x05_Pin, U1 ATtiny202-SS

Commit message: 回路図のリファクタリング
Parts:
- removed the 470 at (118.4, 62.2)
- removed the 470 at (139.4, 126.7)
- removed the 470 at (76.4, 110.5)
- removed the 470 at (97.4, 78.3)
- removed the 470 at (139.4, 62.2)
- removed the 470 at (97.4, 126.7)
- removed the 470 at (139.4, 94.5)
- removed the 470 at (139.4, 110.5)
- removed the 470 at (118.4, 78.3)
- removed the 470 at (76.4, 94.5)
- removed the 470 at (76.4, 62.2)
- removed the 470 at (97.4, 110.5)
- removed the 470 at (118.4, 94.5)
- removed the 470 at (118.4, 126.7)
- removed the 470 at (97.4, 62.2)
- removed the 470 at (76.4, 126.7)
- removed the 470 at (139.4, 78.3)
- removed the 470 at (118.4, 110.5)
- removed the 470 at (97.4, 94.5)
- removed the 470 at (76.4, 78.3)
- removed the D3 at (100.0, 78.0)
- removed the D3 at (142.0, 126.2)
- removed the D3 at (100.0, 126.2)
- removed the D3 at (100.0, 110.2)
- removed the D3 at (142.0, 110.2)
- removed the D3 at (121.0, 126.2)
- removed the D3 at (100.0, 94.0)
- removed the D3 at (79.0, 61.9)
- removed the D3 at (121.0, 94.0)
- removed the D3 at (79.0, 78.0)
- removed the D3 at (142.0, 94.0)
- removed the D3 at (100.0, 61.9)
- removed the D3 at (142.0, 78.0)
- removed the D3 at (79.0, 110.2)
- removed the D3 at (121.0, 61.9)
- removed the D3 at (121.0, 110.2)
- removed the D3 at (79.0, 126.2)
- removed the D3 at (142.0, 61.9)
- removed the D3 at (121.0, 78.0)
- removed the D3 at (79.0, 94.0)
- removed the J1 at (88.5, 125.5)
- removed the J1 at (109.5, 93.3)
- removed the J1 at (130.6, 125.5)
- removed the J1 at (109.5, 125.5)
- removed the J1 at (88.5, 93.3)
- removed the J1 at (88.5, 77.2)
- removed the J1 at (130.6, 61.1)
- removed the J1 at (109.5, 77.2)
- removed the J1 at (67.5, 77.2)
- removed the J1 at (109.5, 61.1)
- removed the J1 at (130.6, 109.5)
- removed the J1 at (130.6, 77.2)
- removed the J1 at (88.5, 109.5)
- removed the J1 at (88.5, 61.1)
- removed the J1 at (109.5, 109.5)
- removed the J1 at (67.5, 109.5)
- removed the J1 at (67.5, 125.5)
- removed the J1 at (67.5, 93.3)
- removed the J1 at (130.6, 93.3)
- removed the J1 at (67.5, 61.1)
- removed the J2 at (82.6, 93.3)
- removed the J2 at (145.6, 93.3)
- removed the J2 at (124.6, 125.5)
- removed the J2 at (124.6, 109.5)
- removed the J2 at (124.6, 93.3)
- removed the J2 at (103.6, 109.5)
- removed the J2 at (82.6, 109.5)
- removed the J2 at (145.6, 125.5)
- removed the J2 at (82.6, 61.1)
- removed the J2 at (103.6, 125.5)
- removed the J2 at (124.6, 61.1)
- removed the J2 at (103.6, 61.1)
- removed the J2 at (103.6, 93.3)
- removed the J2 at (103.6, 77.2)
- removed the J2 at (124.6, 77.2)
- removed the J2 at (145.6, 61.1)
- removed the J2 at (145.6, 109.5)
- removed the J2 at (145.6, 77.2)
- removed the J2 at (82.6, 77.2)
- removed the J2 at (82.6, 125.5)
- removed the LED1 at (92.5, 104.1)
- removed the LED1 at (134.6, 71.9)
- removed the LED1 at (92.5, 136.3)
- removed the LED1 at (134.6, 136.3)
- removed the LED1 at (71.5, 104.1)
- removed the LED1 at (134.6, 104.1)
- removed the LED1 at (113.5, 136.3)
- removed the LED1 at (71.5, 88.0)
- removed the LED1 at (113.5, 71.9)
- removed the LED1 at (113.5, 88.0)
- removed the LED1 at (71.5, 136.3)
- removed the LED1 at (134.6, 88.0)
- removed the LED1 at (71.5, 120.2)
- removed the LED1 at (113.5, 120.2)
- removed the LED1 at (134.6, 120.2)
- removed the LED1 at (92.5, 71.9)
- removed the LED1 at (113.5, 104.1)
- removed the LED1 at (71.5, 71.9)
- removed the LED1 at (92.5, 120.2)
- removed the LED1 at (92.5, 88.0)
- removed the LED2 at (133.8, 109.8)
- removed the LED2 at (70.8, 109.8)
- removed the LED2 at (70.8, 125.8)
- removed the LED2 at (112.8, 125.8)
- removed the LED2 at (91.8, 109.8)
- removed the LED2 at (133.8, 61.5)
- removed the LED2 at (91.8, 93.7)
- removed the LED2 at (112.8, 109.8)
- removed the LED2 at (112.8, 77.5)
- removed the LED2 at (133.8, 125.8)
- removed the LED2 at (91.8, 77.5)
- removed the LED2 at (70.8, 77.5)
- removed the LED2 at (112.8, 61.5)
- removed the LED2 at (70.8, 93.7)
- removed the LED2 at (70.8, 61.5)
- removed the LED2 at (91.8, 61.5)
- removed the LED2 at (91.8, 125.8)
- removed the LED2 at (112.8, 93.7)
- removed the LED2 at (133.8, 93.7)
- removed the LED2 at (133.8, 77.5)
- removed the R1 at (142.1, 88.0)
- removed the R1 at (121.0, 88.0)
- removed the R1 at (121.0, 104.1)
- removed the R1 at (142.1, 104.1)
- removed the R1 at (142.1, 71.9)
- removed the R1 at (79.0, 88.0)
- removed the R1 at (121.0, 71.9)
- removed the R1 at (79.0, 104.1)
- removed the R1 at (79.0, 136.3)
- removed the R1 at (100.0, 120.2)
- removed the R1 at (142.1, 136.3)
- removed the R1 at (79.0, 120.2)
- removed the R1 at (121.0, 120.2)
- removed the R1 at (100.0, 136.3)
- removed the R1 at (79.0, 71.9)
- removed the R1 at (142.1, 120.2)
- removed the R1 at (100.0, 104.1)
- removed the R1 at (100.0, 88.0)
- removed the R1 at (100.0, 71.9)
- removed the R1 at (121.0, 136.3)
- removed the R2 at (136.6, 61.4)
- removed the R2 at (115.5, 61.4)
- removed the R2 at (136.6, 77.5)
- removed the R2 at (73.5, 93.6)
- removed the R2 at (73.5, 61.4)
- removed the R2 at (73.5, 125.8)
- removed the R2 at (94.5, 77.5)
- removed the R2 at (94.5, 61.4)
- removed the R2 at (94.5, 93.6)
- removed the R2 at (73.5, 109.7)
- removed the R2 at (73.5, 77.5)
- removed the R2 at (136.6, 93.6)
- removed the R2 at (136.6, 125.8)
- removed the R2 at (115.5, 77.5)
- removed the R2 at (94.5, 109.7)
- removed the R2 at (115.5, 125.8)
- removed the R2 at (115.5, 93.6)
- removed the R2 at (136.6, 109.7)
- removed the R2 at (94.5, 125.8)
- removed the R2 at (115.5, 109.7)
- removed the U1 at (94.8, 84.0)
- removed the U1 at (136.8, 132.3)
- removed the U1 at (136.8, 84.0)
- removed the U1 at (115.8, 116.2)
- removed the U1 at (73.8, 84.0)
- removed the U1 at (94.8, 67.9)
- removed the U1 at (136.8, 67.9)
- removed the U1 at (115.8, 84.0)
- removed the U1 at (136.8, 116.2)
- removed the U1 at (94.8, 132.3)
- removed the U1 at (94.8, 116.2)
- removed the U1 at (94.8, 100.1)
- removed the U1 at (115.8, 100.1)
- removed the U1 at (115.8, 132.3)
- removed the U1 at (136.8, 100.1)
- removed the U1 at (73.8, 132.3)
- removed the U1 at (115.8, 67.9)
- removed the U1 at (73.8, 116.2)
- removed the U1 at (73.8, 67.9)
- removed the U1 at (73.8, 100.1)
- added 470: R3, Resistor_SMD:R_0603_1608Metric, F.Cu at (269.8, 94.5)
- added 470: R3, Resistor_SMD:R_0603_1608Metric, F.Cu at (248.8, 94.5)
- added 470: R3, Resistor_SMD:R_0603_1608Metric, F.Cu at (290.8, 46.2)
- added 470: R3, Resistor_SMD:R_0603_1608Metric, F.Cu at (248.8, 46.2)
- added 470: R3, Resistor_SMD:R_0603_1608Metric, F.Cu at (290.8, 30.1)
- added 470: R3, Resistor_SMD:R_0603_1608Metric, F.Cu at (248.8, 62.4)
- added 470: R3, Resistor_SMD:R_0603_1608Metric, F.Cu at (227.8, 94.5)
- added 470: R3, Resistor_SMD:R_0603_1608Metric, F.Cu at (290.8, 78.5)
- added 470: R3, Resistor_SMD:R_0603_1608Metric, F.Cu at (290.8, 94.5)
- added 470: R3, Resistor_SMD:R_0603_1608Metric, F.Cu at (290.8, 62.4)
- added 470: R3, Resistor_SMD:R_0603_1608Metric, F.Cu at (227.8, 30.1)
- added 470: R3, Resistor_SMD:R_0603_1608Metric, F.Cu at (269.8, 30.1)
- added 470: R3, Resistor_SMD:R_0603_1608Metric, F.Cu at (248.8, 30.1)
- added 470: R3, Resistor_SMD:R_0603_1608Metric, F.Cu at (227.8, 62.4)
- added 470: R3, Resistor_SMD:R_0603_1608Metric, F.Cu at (227.8, 78.5)
- added 470: R3, Resistor_SMD:R_0603_1608Metric, F.Cu at (269.8, 46.2)
- added 470: R3, Resistor_SMD:R_0603_1608Metric, F.Cu at (248.8, 78.5)
- added 470: R3, Resistor_SMD:R_0603_1608Metric, F.Cu at (269.8, 78.5)
- added 470: R3, Resistor_SMD:R_0603_1608Metric, F.Cu at (269.8, 62.4)
- added 470: R3, Resistor_SMD:R_0603_1608Metric, F.Cu at (227.8, 46.2)
- added D3: RB160M-30, Diode_SMD:D_1206_3216Metric, F.Cu at (293.4, 29.8)
- added D3: RB160M-30, Diode_SMD:D_1206_3216Metric, F.Cu at (230.4, 62.0)
- added D3: RB160M-30, Diode_SMD:D_1206_3216Metric, F.Cu at (272.4, 62.0)
- added D3: RB160M-30, Diode_SMD:D_1206_3216Metric, F.Cu at (272.4, 45.9)
- added D3: RB160M-30, Diode_SMD:D_1206_3216Metric, F.Cu at (272.4, 78.0)
- added D3: RB160M-30, Diode_SMD:D_1206_3216Metric, F.Cu at (230.4, 45.9)
- added D3: RB160M-30, Diode_SMD:D_1206_3216Metric, F.Cu at (251.4, 94.2)
- added D3: RB160M-30, Diode_SMD:D_1206_3216Metric, F.Cu at (251.4, 78.0)
- added D3: RB160M-30, Diode_SMD:D_1206_3216Metric, F.Cu at (272.4, 94.2)
- added D3: RB160M-30, Diode_SMD:D_1206_3216Metric, F.Cu at (251.4, 29.8)
- added D3: RB160M-30, Diode_SMD:D_1206_3216Metric, F.Cu at (293.4, 78.0)
- added D3: RB160M-30, Diode_SMD:D_1206_3216Metric, F.Cu at (293.4, 45.9)
- added D3: RB160M-30, Diode_SMD:D_1206_3216Metric, F.Cu at (230.4, 29.8)
- added D3: RB160M-30, Diode_SMD:D_1206_3216Metric, F.Cu at (251.4, 45.9)
- added D3: RB160M-30, Diode_SMD:D_1206_3216Metric, F.Cu at (272.4, 29.8)
- added D3: RB160M-30, Diode_SMD:D_1206_3216Metric, F.Cu at (230.4, 94.2)
- added D3: RB160M-30, Diode_SMD:D_1206_3216Metric, F.Cu at (293.4, 62.0)
- added D3: RB160M-30, Diode_SMD:D_1206_3216Metric, F.Cu at (230.4, 78.0)
- added D3: RB160M-30, Diode_SMD:D_1206_3216Metric, F.Cu at (251.4, 62.0)
- added D3: RB160M-30, Diode_SMD:D_1206_3216Metric, F.Cu at (293.4, 94.2)
- added J1: Conn_01x05_Pin, Connector_PinHeader_2.54mm:PinHeader_1x05_P2.54mm_Vertical, B.Cu at (260.9, 29.1)
- added J1: Conn_01x05_Pin, Connector_PinHeader_2.54mm:PinHeader_1x05_P2.54mm_Vertical, B.Cu at (260.9, 45.1)
- added J1: Conn_01x05_Pin, Connector_PinHeader_2.54mm:PinHeader_1x05_P2.54mm_Vertical, B.Cu at (218.9, 93.5)
- added J1: Conn_01x05_Pin, Connector_PinHeader_2.54mm:PinHeader_1x05_P2.54mm_Vertical, B.Cu at (260.9, 61.2)
- added J1: Conn_01x05_Pin, Connector_PinHeader_2.54mm:PinHeader_1x05_P2.54mm_Vertical, B.Cu at (239.9, 45.1)
- added J1: Conn_01x05_Pin, Connector_PinHeader_2.54mm:PinHeader_1x05_P2.54mm_Vertical, B.Cu at (218.9, 29.1)
- added J1: Conn_01x05_Pin, Connector_PinHeader_2.54mm:PinHeader_1x05_P2.54mm_Vertical, B.Cu at (281.9, 93.5)
- added J1: Conn_01x05_Pin, Connector_PinHeader_2.54mm:PinHeader_1x05_P2.54mm_Vertical, B.Cu at (218.9, 61.2)
- added J1: Conn_01x05_Pin, Connector_PinHeader_2.54mm:PinHeader_1x05_P2.54mm_Vertical, B.Cu at (239.9, 93.5)
- added J1: Conn_01x05_Pin, Connector_PinHeader_2.54mm:PinHeader_1x05_P2.54mm_Vertical, B.Cu at (281.9, 77.3)
- added J1: Conn_01x05_Pin, Connector_PinHeader_2.54mm:PinHeader_1x05_P2.54mm_Vertical, B.Cu at (260.9, 93.5)
- added J1: Conn_01x05_Pin, Connector_PinHeader_2.54mm:PinHeader_1x05_P2.54mm_Vertical, B.Cu at (260.9, 77.3)
- added J1: Conn_01x05_Pin, Connector_PinHeader_2.54mm:PinHeader_1x05_P2.54mm_Vertical, B.Cu at (239.9, 61.2)
- added J1: Conn_01x05_Pin, Connector_PinHeader_2.54mm:PinHeader_1x05_P2.54mm_Vertical, B.Cu at (239.9, 77.3)
- added J1: Conn_01x05_Pin, Connector_PinHeader_2.54mm:PinHeader_1x05_P2.54mm_Vertical, B.Cu at (239.9, 29.1)
- added J1: Conn_01x05_Pin, Connector_PinHeader_2.54mm:PinHeader_1x05_P2.54mm_Vertical, B.Cu at (218.9, 45.1)
- added J1: Conn_01x05_Pin, Connector_PinHeader_2.54mm:PinHeader_1x05_P2.54mm_Vertical, B.Cu at (281.9, 29.1)
- added J1: Conn_01x05_Pin, Connector_PinHeader_2.54mm:PinHeader_1x05_P2.54mm_Vertical, B.Cu at (281.9, 45.1)
- added J1: Conn_01x05_Pin, Connector_PinHeader_2.54mm:PinHeader_1x05_P2.54mm_Vertical, B.Cu at (281.9, 61.2)
- added J1: Conn_01x05_Pin, Connector_PinHeader_2.54mm:PinHeader_1x05_P2.54mm_Vertical, B.Cu at (218.9, 77.3)
- added J2: Conn_01x05_Pin, Connector_PinHeader_2.54mm:PinHeader_1x05_P2.54mm_Vertical, B.Cu at (255.0, 93.5)
- added J2: Conn_01x05_Pin, Connector_PinHeader_2.54mm:PinHeader_1x05_P2.54mm_Vertical, B.Cu at (276.0, 61.2)
- added J2: Conn_01x05_Pin, Connector_PinHeader_2.54mm:PinHeader_1x05_P2.54mm_Vertical, B.Cu at (255.0, 77.3)
- added J2: Conn_01x05_Pin, Connector_PinHeader_2.54mm:PinHeader_1x05_P2.54mm_Vertical, B.Cu at (234.0, 29.1)
- added J2: Conn_01x05_Pin, Connector_PinHeader_2.54mm:PinHeader_1x05_P2.54mm_Vertical, B.Cu at (297.0, 77.3)
- added J2: Conn_01x05_Pin, Connector_PinHeader_2.54mm:PinHeader_1x05_P2.54mm_Vertical, B.Cu at (297.0, 61.2)
- added J2: Conn_01x05_Pin, Connector_PinHeader_2.54mm:PinHeader_1x05_P2.54mm_Vertical, B.Cu at (297.0, 29.1)
- added J2: Conn_01x05_Pin, Connector_PinHeader_2.54mm:PinHeader_1x05_P2.54mm_Vertical, B.Cu at (297.0, 93.5)
- added J2: Conn_01x05_Pin, Connector_PinHeader_2.54mm:PinHeader_1x05_P2.54mm_Vertical, B.Cu at (276.0, 45.1)
- added J2: Conn_01x05_Pin, Connector_PinHeader_2.54mm:PinHeader_1x05_P2.54mm_Vertical, B.Cu at (255.0, 45.1)
- added J2: Conn_01x05_Pin, Connector_PinHeader_2.54mm:PinHeader_1x05_P2.54mm_Vertical, B.Cu at (234.0, 61.2)
- added J2: Conn_01x05_Pin, Connector_PinHeader_2.54mm:PinHeader_1x05_P2.54mm_Vertical, B.Cu at (276.0, 29.1)
- added J2: Conn_01x05_Pin, Connector_PinHeader_2.54mm:PinHeader_1x05_P2.54mm_Vertical, B.Cu at (234.0, 45.1)
- added J2: Conn_01x05_Pin, Connector_PinHeader_2.54mm:PinHeader_1x05_P2.54mm_Vertical, B.Cu at (234.0, 77.3)
- added J2: Conn_01x05_Pin, Connector_PinHeader_2.54mm:PinHeader_1x05_P2.54mm_Vertical, B.Cu at (297.0, 45.1)
- added J2: Conn_01x05_Pin, Connector_PinHeader_2.54mm:PinHeader_1x05_P2.54mm_Vertical, B.Cu at (234.0, 93.5)
- added J2: Conn_01x05_Pin, Connector_PinHeader_2.54mm:PinHeader_1x05_P2.54mm_Vertical, B.Cu at (276.0, 77.3)
- added J2: Conn_01x05_Pin, Connector_PinHeader_2.54mm:PinHeader_1x05_P2.54mm_Vertical, B.Cu at (255.0, 29.1)
- added J2: Conn_01x05_Pin, Connector_PinHeader_2.54mm:PinHeader_1x05_P2.54mm_Vertical, B.Cu at (276.0, 93.5)
- added J2: Conn_01x05_Pin, Connector_PinHeader_2.54mm:PinHeader_1x05_P2.54mm_Vertical, B.Cu at (255.0, 61.2)
- added LED1: LED_G, Diode_SMD:D_0603_1608Metric, F.Cu at (285.9, 72.0)
- added LED1: LED_G, Diode_SMD:D_0603_1608Metric, F.Cu at (264.9, 55.9)
- added LED1: LED_G, Diode_SMD:D_0603_1608Metric, F.Cu at (264.9, 104.2)
- added LED1: LED_G, Diode_SMD:D_0603_1608Metric, F.Cu at (243.9, 55.9)
- added LED1: LED_G, Diode_SMD:D_0603_1608Metric, F.Cu at (222.9, 104.2)
- added LED1: LED_G, Diode_SMD:D_0603_1608Metric, F.Cu at (285.9, 88.1)
- added LED1: LED_G, Diode_SMD:D_0603_1608Metric, F.Cu at (243.9, 39.8)
- added LED1: LED_G, Diode_SMD:D_0603_1608Metric, F.Cu at (243.9, 104.2)
- added LED1: LED_G, Diode_SMD:D_0603_1608Metric, F.Cu at (264.9, 72.0)
- added LED1: LED_G, Diode_SMD:D_0603_1608Metric, F.Cu at (243.9, 72.0)
- added LED1: LED_G, Diode_SMD:D_0603_1608Metric, F.Cu at (264.9, 39.8)
- added LED1: LED_G, Diode_SMD:D_0603_1608Metric, F.Cu at (285.9, 39.8)
- added LED1: LED_G, Diode_SMD:D_0603_1608Metric, F.Cu at (222.9, 72.0)
- added LED1: LED_G, Diode_SMD:D_0603_1608Metric, F.Cu at (222.9, 55.9)
- added LED1: LED_G, Diode_SMD:D_0603_1608Metric, F.Cu at (222.9, 39.8)
- added LED1: LED_G, Diode_SMD:D_0603_1608Metric, F.Cu at (285.9, 55.9)
- added LED1: LED_G, Diode_SMD:D_0603_1608Metric, F.Cu at (264.9, 88.1)
- added LED1: LED_G, Diode_SMD:D_0603_1608Metric, F.Cu at (222.9, 88.1)
- added LED1: LED_G, Diode_SMD:D_0603_1608Metric, F.Cu at (285.9, 104.2)
- added LED1: LED_G, Diode_SMD:D_0603_1608Metric, F.Cu at (243.9, 88.1)
- added LED2: LED_R, Diode_SMD:D_0603_1608Metric, F.Cu at (285.2, 29.4)
- added LED2: LED_R, Diode_SMD:D_0603_1608Metric, F.Cu at (264.2, 77.7)
- added LED2: LED_R, Diode_SMD:D_0603_1608Metric, F.Cu at (222.2, 29.4)
- added LED2: LED_R, Diode_SMD:D_0603_1608Metric, F.Cu at (285.2, 93.8)
- added LED2: LED_R, Diode_SMD:D_0603_1608Metric, F.Cu at (243.2, 77.7)
- added LED2: LED_R, Diode_SMD:D_0603_1608Metric, F.Cu at (243.2, 45.5)
- added LED2: LED_R, Diode_SMD:D_0603_1608Metric, F.Cu at (285.2, 45.5)
- added LED2: LED_R, Diode_SMD:D_0603_1608Metric, F.Cu at (285.2, 61.5)
- added LED2: LED_R, Diode_SMD:D_0603_1608Metric, F.Cu at (222.2, 45.5)
- added LED2: LED_R, Diode_SMD:D_0603_1608Metric, F.Cu at (243.2, 93.8)
- added LED2: LED_R, Diode_SMD:D_0603_1608Metric, F.Cu at (285.2, 77.7)
- added LED2: LED_R, Diode_SMD:D_0603_1608Metric, F.Cu at (243.2, 61.5)
- added LED2: LED_R, Diode_SMD:D_0603_1608Metric, F.Cu at (222.2, 93.8)
- added LED2: LED_R, Diode_SMD:D_0603_1608Metric, F.Cu at (264.2, 45.5)
- added LED2: LED_R, Diode_SMD:D_0603_1608Metric, F.Cu at (243.2, 29.4)
- added LED2: LED_R, Diode_SMD:D_0603_1608Metric, F.Cu at (222.2, 61.5)
- added LED2: LED_R, Diode_SMD:D_0603_1608Metric, F.Cu at (264.2, 93.8)
- added LED2: LED_R, Diode_SMD:D_0603_1608Metric, F.Cu at (222.2, 77.7)
- added LED2: LED_R, Diode_SMD:D_0603_1608Metric, F.Cu at (264.2, 61.5)
- added LED2: LED_R, Diode_SMD:D_0603_1608Metric, F.Cu at (264.2, 29.4)
- added R1: 1k, Resistor_SMD:R_0603_1608Metric, F.Cu at (293.4, 72.0)
- added R1: 1k, Resistor_SMD:R_0603_1608Metric, F.Cu at (230.4, 88.1)
- added R1: 1k, Resistor_SMD:R_0603_1608Metric, F.Cu at (230.4, 39.8)
- added R1: 1k, Resistor_SMD:R_0603_1608Metric, F.Cu at (293.4, 55.9)
- added R1: 1k, Resistor_SMD:R_0603_1608Metric, F.Cu at (272.4, 55.9)
- added R1: 1k, Resistor_SMD:R_0603_1608Metric, F.Cu at (293.4, 88.1)
- added R1: 1k, Resistor_SMD:R_0603_1608Metric, F.Cu at (230.4, 104.2)
- added R1: 1k, Resistor_SMD:R_0603_1608Metric, F.Cu at (251.4, 55.9)
- added R1: 1k, Resistor_SMD:R_0603_1608Metric, F.Cu at (293.4, 39.8)
- added R1: 1k, Resistor_SMD:R_0603_1608Metric, F.Cu at (251.4, 104.2)
- added R1: 1k, Resistor_SMD:R_0603_1608Metric, F.Cu at (272.4, 104.2)
- added R1: 1k, Resistor_SMD:R_0603_1608Metric, F.Cu at (230.4, 72.0)
- added R1: 1k, Resistor_SMD:R_0603_1608Metric, F.Cu at (293.4, 104.2)
- added R1: 1k, Resistor_SMD:R_0603_1608Metric, F.Cu at (251.4, 72.0)
- added R1: 1k, Resistor_SMD:R_0603_1608Metric, F.Cu at (251.4, 39.8)
- added R1: 1k, Resistor_SMD:R_0603_1608Metric, F.Cu at (272.4, 88.1)
- added R1: 1k, Resistor_SMD:R_0603_1608Metric, F.Cu at (230.4, 55.9)
- added R1: 1k, Resistor_SMD:R_0603_1608Metric, F.Cu at (272.4, 39.8)
- added R1: 1k, Resistor_SMD:R_0603_1608Metric, F.Cu at (251.4, 88.1)
- added R1: 1k, Resistor_SMD:R_0603_1608Metric, F.Cu at (272.4, 72.0)
- added R2: 1k, Resistor_SMD:R_0603_1608Metric, F.Cu at (266.9, 93.7)
- added R2: 1k, Resistor_SMD:R_0603_1608Metric, F.Cu at (287.9, 61.5)
- added R2: 1k, Resistor_SMD:R_0603_1608Metric, F.Cu at (245.9, 29.3)
- added R2: 1k, Resistor_SMD:R_0603_1608Metric, F.Cu at (287.9, 77.6)
- added R2: 1k, Resistor_SMD:R_0603_1608Metric, F.Cu at (245.9, 77.6)
- added R2: 1k, Resistor_SMD:R_0603_1608Metric, F.Cu at (245.9, 61.5)
- added R2: 1k, Resistor_SMD:R_0603_1608Metric, F.Cu at (224.9, 29.3)
- added R2: 1k, Resistor_SMD:R_0603_1608Metric, F.Cu at (287.9, 29.3)
- added R2: 1k, Resistor_SMD:R_0603_1608Metric, F.Cu at (266.9, 45.4)
- added R2: 1k, Resistor_SMD:R_0603_1608Metric, F.Cu at (224.9, 77.6)
- added R2: 1k, Resistor_SMD:R_0603_1608Metric, F.Cu at (287.9, 93.7)
- added R2: 1k, Resistor_SMD:R_0603_1608Metric, F.Cu at (245.9, 45.4)
- added R2: 1k, Resistor_SMD:R_0603_1608Metric, F.Cu at (266.9, 77.6)
- added R2: 1k, Resistor_SMD:R_0603_1608Metric, F.Cu at (245.9, 93.7)
- added R2: 1k, Resistor_SMD:R_0603_1608Metric, F.Cu at (266.9, 61.5)
- added R2: 1k, Resistor_SMD:R_0603_1608Metric, F.Cu at (287.9, 45.4)
- added R2: 1k, Resistor_SMD:R_0603_1608Metric, F.Cu at (224.9, 61.5)
- added R2: 1k, Resistor_SMD:R_0603_1608Metric, F.Cu at (224.9, 93.7)
- added R2: 1k, Resistor_SMD:R_0603_1608Metric, F.Cu at (224.9, 45.4)
- added R2: 1k, Resistor_SMD:R_0603_1608Metric, F.Cu at (266.9, 29.3)
- added U1: ATtiny202-SS, Package_SO:SOIC-8_3.9x4.9mm_P1.27mm, F.Cu at (267.2, 100.2)
- added U1: ATtiny202-SS, Package_SO:SOIC-8_3.9x4.9mm_P1.27mm, F.Cu at (288.2, 84.1)
- added U1: ATtiny202-SS, Package_SO:SOIC-8_3.9x4.9mm_P1.27mm, F.Cu at (288.2, 51.9)
- added U1: ATtiny202-SS, Package_SO:SOIC-8_3.9x4.9mm_P1.27mm, F.Cu at (246.2, 100.2)
- added U1: ATtiny202-SS, Package_SO:SOIC-8_3.9x4.9mm_P1.27mm, F.Cu at (246.2, 51.9)
- added U1: ATtiny202-SS, Package_SO:SOIC-8_3.9x4.9mm_P1.27mm, F.Cu at (225.2, 84.1)
- added U1: ATtiny202-SS, Package_SO:SOIC-8_3.9x4.9mm_P1.27mm, F.Cu at (267.2, 35.8)
- added U1: ATtiny202-SS, Package_SO:SOIC-8_3.9x4.9mm_P1.27mm, F.Cu at (225.2, 51.9)
- added U1: ATtiny202-SS, Package_SO:SOIC-8_3.9x4.9mm_P1.27mm, F.Cu at (267.2, 68.0)
- added U1: ATtiny202-SS, Package_SO:SOIC-8_3.9x4.9mm_P1.27mm, F.Cu at (246.2, 68.0)
- added U1: ATtiny202-SS, Package_SO:SOIC-8_3.9x4.9mm_P1.27mm, F.Cu at (267.2, 84.1)
- added U1: ATtiny202-SS, Package_SO:SOIC-8_3.9x4.9mm_P1.27mm, F.Cu at (225.2, 100.2)
- added U1: ATtiny202-SS, Package_SO:SOIC-8_3.9x4.9mm_P1.27mm, F.Cu at (288.2, 100.2)
- added U1: ATtiny202-SS, Package_SO:SOIC-8_3.9x4.9mm_P1.27mm, F.Cu at (288.2, 68.0)
- added U1: ATtiny202-SS, Package_SO:SOIC-8_3.9x4.9mm_P1.27mm, F.Cu at (225.2, 35.8)
- added U1: ATtiny202-SS, Package_SO:SOIC-8_3.9x4.9mm_P1.27mm, F.Cu at (225.2, 68.0)
- added U1: ATtiny202-SS, Package_SO:SOIC-8_3.9x4.9mm_P1.27mm, F.Cu at (288.2, 35.8)
- added U1: ATtiny202-SS, Package_SO:SOIC-8_3.9x4.9mm_P1.27mm, F.Cu at (246.2, 84.1)
- added U1: ATtiny202-SS, Package_SO:SOIC-8_3.9x4.9mm_P1.27mm, F.Cu at (246.2, 35.8)
- added U1: ATtiny202-SS, Package_SO:SOIC-8_3.9x4.9mm_P1.27mm, F.Cu at (267.2, 51.9)
- moved KiKit_MB_10_3 154.8 mm to (278.2, 32.3)
- moved KiKit_MB_10_4 154.8 mm to (278.2, 33.2)
- moved KiKit_MB_10_5 154.8 mm to (278.2, 34.0)
- moved KiKit_MB_10_6 154.8 mm to (278.2, 34.9)
- moved KiKit_MB_10_7 154.8 mm to (278.2, 35.8)
- moved KiKit_MB_11_3 154.8 mm to (266.8, 26.8)
- moved KiKit_MB_11_4 154.8 mm to (267.6, 26.8)
- moved KiKit_MB_11_5 154.8 mm to (268.5, 26.8)
- moved KiKit_MB_11_6 154.8 mm to (269.4, 26.8)
- moved KiKit_MB_11_7 154.8 mm to (270.2, 26.8)
- moved KiKit_MB_12_3 154.8 mm to (270.2, 41.4)
- moved KiKit_MB_12_4 154.8 mm to (269.4, 41.4)
- moved KiKit_MB_12_5 154.8 mm to (268.5, 41.4)
- moved KiKit_MB_12_6 154.8 mm to (267.6, 41.4)
- moved KiKit_MB_12_7 154.8 mm to (266.8, 41.4)
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Routing:
- net Board_13-Net-(LED1-K): track 0.00 -> 8.18 mm
- net Board_12-Net-(LED1-K): track 0.00 -> 8.18 mm
- net Board_11-Net-(D1-K): track 8.18 -> 0.00 mm
- net Board_1-Net-(LED1-K): track 0.00 -> 8.18 mm
- net Board_0-Net-(LED1-K): track 0.00 -> 8.18 mm
- net Board_4-Net-(LED1-K): track 0.00 -> 8.18 mm
- net Board_5-Net-(LED1-K): track 0.00 -> 8.18 mm
- net Board_9-Net-(D1-K): track 8.18 -> 0.00 mm
- net Board_8-Net-(D1-K): track 8.18 -> 0.00 mm
- net Board_10-Net-(D1-K): track 8.18 -> 0.00 mm
- net Board_9-Net-(LED1-K): track 0.00 -> 8.18 mm
- net Board_8-Net-(LED1-K): track 0.00 -> 8.18 mm
- net Board_15-Net-(LED1-K): track 0.00 -> 8.18 mm
- net Board_14-Net-(LED1-K): track 0.00 -> 8.18 mm
- net Board_17-Net-(LED1-K): track 0.00 -> 8.18 mm
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Other:
- outline, holes or cut-outs redrawn
