File: pcb/tinypico.kicad_sch (KiCad schematic)
At the start: 9 parts, among them J1 Conn_01x05_Pin, J2 Conn_01x05_Pin, U1 ATtiny202-SS

Commit message: RXとTXを入れ替え。他リファクタリング。
Parts:
- LED1: renamed from D1; value LED -> LED_G
- LED2: renamed from D2; value LED -> LED_R
Connections:
- net UPDI_RX: now also D3.1 (K); no longer D3.2 (A), R3.2
- net UPDI_TX: now also D3.2 (A), R3.2; no longer D3.1 (K)
Other:
- note added: "※ UPDI_TX <--> USB_serial_RX UPDI_RX <--> USB_serial_TX"
Changed lines of the file:
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@@
     (effects (font (size 1.6 1.6)) (justify left bottom))
+  )
+  (text "※ UPDI_TX <--> USB_serial_RX\n   UPDI_RX <--> USB_serial_TX"
+    (at 142.24 26.67 0)
+    (effects (font (size 1.27 1.27)) (justify right bottom))
   )
   (text "Cost\nATtiny202 JPY70\n1608 LED G JPY10\n1608 LED R JPY14\n1608 Resister 1k JPY20 x2\n1608 Resister 470 JPY20\nDiode RB160M-B JPY15\nPINHEADER JPY2\nPCB JPY20"
@@
     )
   )
-  (global_label "UPDI_RX" (shape input) (at 115.57 43.18 0) (fields_autoplaced)
-    (effects (font (size 1.27 1.27)) (justify left))
-    (property "Intersheetrefs" "${INTERSHEET_REFS}" (at 126.4776 43.18 0)
+  (global_label "UPDI_TX" (shape input) (at 115.57 43.18 0) (fields_autoplaced)
+    (effects (font (size 1.27 1.27)) (justify left))
+    (property "Intersheetrefs" "${INTERSHEET_REFS}" (at 126.1752 43.18 0)
       (effects (font (size 1.27 1.27)) (justify left) hide)
     )
@@
     )
   )
-  (global_label "UPDI_TX" (shape input) (at 115.57 36.83 0) (fields_autoplaced)
-    (effects (font (size 1.27 1.27)) (justify left))
-    (property "Intersheetrefs" "${INTERSHEET_REFS}" (at 126.1752 36.83 0)
+  (global_label "UPDI_RX" (shape input) (at 115.57 36.83 0) (fields_autoplaced)
+    (effects (font (size 1.27 1.27)) (justify left))
+    (property "Intersheetrefs" "${INTERSHEET_REFS}" (at 126.4776 36.83 0)
       (effects (font (size 1.27 1.27)) (justify left) hide)
     )
@@
   (symbol (lib_id "Device:LED") (at 31.75 39.37 90) (unit 1)
     (in_bom yes) (on_board yes) (dnp no) (fields_autoplaced)
-    (property "Reference" "D2" (at 35.56 39.6875 90)
+    (property "Reference" "LED2" (at 35.56 39.6875 90)
       (effects (font (size 1.27 1.27)) (justify right))
     )
-    (property "Value" "LED" (at 35.56 42.2275 90)
+    (property "Value" "LED_R" (at 35.56 42.2275 90)
       (effects (font (size 1.27 1.27)) (justify right))
     )
@@
       (project "tinypico"
         (path "/0702e63e-4e25-4f10-b02c-41d44a9420fc"
-          (reference "D2") (unit 1)
+          (reference "LED2") (unit 1)
         )
       )
@@
   (symbol (lib_id "Device:LED") (at 95.25 68.58 180) (unit 1)
     (in_bom yes) (on_board yes) (dnp no)
-    (property "Reference" "D1" (at 96.52 71.12 0)
-      (effects (font (size 1.27 1.27)))
-    )
-    (property "Value" "LED" (at 96.52 73.66 0)
+    (property "Reference" "LED1" (at 96.52 71.12 0)
+      (effects (font (size 1.27 1.27)))
+    )
+    (property "Value" "LED_G" (at 96.52 73.66 0)
       (effects (font (size 1.27 1.27)))
     )
@@
       (project "tinypico"
         (path "/0702e63e-4e25-4f10-b02c-41d44a9420fc"
-          (reference "D1") (unit 1)
-        )
-      )
+          (reference "LED1") (unit 1)
+        )
+      )

Commit message: 回路図の誤記訂正
Other:
- note added: "※ UPDI_TX <--> USB_serial_TX UPDI_RX <--> USB_serial_RX"
- note removed: "※ UPDI_TX <--> USB_serial_RX UPDI_RX <--> USB_serial_TX"
Changed lines of the file:
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@@
     (effects (font (size 1.6 1.6)) (justify left bottom))
   )
-  (text "※ UPDI_TX <--> USB_serial_RX\n   UPDI_RX <--> USB_serial_TX"
+  (text "※ UPDI_TX <--> USB_serial_TX\n   UPDI_RX <--> USB_serial_RX"
     (at 142.24 26.67 0)
     (effects (font (size 1.27 1.27)) (justify right bottom))

Commit message: 回路図のリファクタリング
Connections:
- net UPDI_RX: now also D3.2 (A), R3.2; no longer D3.1 (K)
- net UPDI_TX: now also D3.1 (K); no longer D3.2 (A), R3.2
Changed lines of the file:
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@@
     )
   )
-  (global_label "UPDI_TX" (shape input) (at 115.57 43.18 0) (fields_autoplaced)
+  (global_label "UPDI_RX" (shape input) (at 115.57 43.18 0) (fields_autoplaced)
     (effects (font (size 1.27 1.27)) (justify left))
-    (property "Intersheetrefs" "${INTERSHEET_REFS}" (at 126.1752 43.18 0)
+    (property "Intersheetrefs" "${INTERSHEET_REFS}" (at 126.4776 43.18 0)
       (effects (font (size 1.27 1.27)) (justify left) hide)
     )
@@
     )
   )
-  (global_label "UPDI_RX" (shape input) (at 115.57 36.83 0) (fields_autoplaced)
+  (global_label "UPDI_TX" (shape input) (at 115.57 36.83 0) (fields_autoplaced)
     (effects (font (size 1.27 1.27)) (justify left))
-    (property "Intersheetrefs" "${INTERSHEET_REFS}" (at 126.4776 36.83 0)
+    (property "Intersheetrefs" "${INTERSHEET_REFS}" (at 126.1752 36.83 0)
       (effects (font (size 1.27 1.27)) (justify left) hide)
     )

Commit message: リポジトリ名称を変更
Other:
- title: TinyPico -> Tibicon
Changed lines of the file:
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@@
   (paper "A5")
   (title_block
-    (title "TinyPico")
+    (title "Tibicon")
     (date "2024-07-16")
     (rev "1")
